Commit message: Prevent SO101 arm from going limp in Gazebo

File: so101_description/urdf/robots/gz_macro.xacro (robot description, xacro)
@@ -11,3 +11,8 @@
     </gazebo>
   </xacro:macro>
+  <xacro:macro name="gazebo_disable_gravity" params="link_name">
+    <gazebo reference="${link_name}">
+      <gravity>false</gravity>
+    </gazebo>
+  </xacro:macro>
 </robot>

File: so101_description/urdf/robots/so101.urdf.xacro (robot description, xacro)
@@ -455,3 +455,9 @@
   <xacro:gazebo_light_blue_material link_name="gripper_link"/>
   <xacro:gazebo_light_blue_material link_name="moving_jaw_so101_v1_link"/>
+  <xacro:gazebo_disable_gravity link_name="shoulder_link"/>
+  <xacro:gazebo_disable_gravity link_name="upper_arm_link"/>
+  <xacro:gazebo_disable_gravity link_name="lower_arm_link"/>
+  <xacro:gazebo_disable_gravity link_name="wrist_link"/>
+  <xacro:gazebo_disable_gravity link_name="gripper_link"/>
+  <xacro:gazebo_disable_gravity link_name="moving_jaw_so101_v1_link"/>
 </robot>
